File: PCB design/GaN_Transistor_Test_Board/GaN_Transistor_Test_Board.kicad_pcb (KiCad board)
At the start: 2 copper layers, 4 parts, among them Q1 IGD70R500D2S

Commit message: PCB update V1
Parts:
- moved Q1 17.1 mm to (143.3, 92.3)
Changed lines of the file:
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@@
 	)
 	(paper "A4")
+	(title_block
+		(date "18.01.2026")
+		(company "eng. Mateusz Witczak")
+	)
 	(layers
 		(0 "F.Cu" signal)
@@
 	(footprint "Footprints:TO-252-3_TabPin4"
 		(layer "F.Cu")
-		(at 140.675 75.4)
+		(at 143.325 92.275)
 		(descr "TO-252 / DPAK SMD package, http://www.infineon.com/cms/en/product/packages/PG-TO252/PG-TO252-3-1/")
 		(tags "DPAK TO-252 DPAK-3 TO-252-3 SOT-428")
