File: PCB design/GaN_Transistor_Test_Board.kicad_pcb (KiCad board)
At the start: 2 copper layers, 4 parts, among them Q1 IGD70R500D2S

Commit message: Layout redesign
Parts:
- removed E1, E2, E3: 1-1337445-0, Footprints:TE_1-1337445-0
- removed Q1: IGD70R500D2S, Footprints:TO-252-3_TabPin4
