File: PCB design/GaN_Transistor_Test_Board.kicad_pcb (KiCad board)
At the start: 2 copper layers, 0 parts

Commit message: PCB_rev1
Parts:
- added D1: 1-1337445-0, Footprints:TE_1-1337445-0, F.Cu at (71.4, 105.7)
- added D2: 1-1337445-0, Footprints:TE_1-1337445-0, F.Cu at (205.8, 119.8)
- added D3: 1-1337445-0, Footprints:TE_1-1337445-0, F.Cu at (71.4, 154.6)
- added D4: 1-1337445-0, Footprints:TE_1-1337445-0, F.Cu at (205.7, 167.4)
- added G1: 1-1337445-0, Footprints:TE_1-1337445-0, F.Cu at (71.4, 122.3)
- added G2: 1-1337445-0, Footprints:TE_1-1337445-0, F.Cu at (205.8, 136.9)
- added G3: 1-1337445-0, Footprints:TE_1-1337445-0, F.Cu at (71.4, 138.0)
- added G4: 1-1337445-0, Footprints:TE_1-1337445-0, F.Cu at (205.6, 151.8)
- added H1: MountingHole, MountingHole:MountingHole_4.3mm_M4, F.Cu at (71.1, 61.8)
- added H2: MountingHole, MountingHole:MountingHole_4.3mm_M4, F.Cu at (205.8, 61.5)
- added H3: MountingHole, MountingHole:MountingHole_4.3mm_M4, F.Cu at (71.3, 197.3)
- added H4: MountingHole, MountingHole:MountingHole_4.3mm_M4, F.Cu at (205.9, 197.4)
- added J1: Conn_01x01, Footprints:CONN1_FCR7350R_CLF, F.Cu at (139.8, 176.9)
- added J2: Conn_01x01, Footprints:CONN1_FCR7350R_CLF, F.Cu at (114.9, 176.8)
- added J3: Conn_01x01, Footprints:CONN1_FCR7350R_CLF, F.Cu at (164.7, 177.0)
- added Q1: IGD70R500D2S, Footprints:IFX-PG-TO252-3N-37-V1, F.Cu at (129.6, 125.0)
- added Q2: IGD70R500D2S, Footprints:IFX-PG-TO252-3N-37-V1, F.Cu at (151.4, 125.0)
- added Q3: IGD70R500D2S, Footprints:IFX-PG-TO252-3N-37-V1, F.Cu at (129.6, 136.9)
- added Q4: IGD70R500D2S, Footprints:IFX-PG-TO252-3N-37-V1, F.Cu at (151.4, 136.9)
- added R1: 100, Footprints:R_LOAD, F.Cu at (92.2, 60.9)
- added R2: 100, Resistor_SMD:R_1206_3216Metric_Pad1.30x1.75mm_HandSolder, F.Cu at (114.9, 122.6)
- added R3: 100, Footprints:R_LOAD, F.Cu at (187.0, 60.7)
- added R4: 100, Resistor_SMD:R_1206_3216Metric_Pad1.30x1.75mm_HandSolder, F.Cu at (167.8, 127.7)
- added R5: 100, Footprints:R_LOAD, F.Cu at (91.1, 199.0)
- added R6: 100, Resistor_SMD:R_1206_3216Metric_Pad1.30x1.75mm_HandSolder, F.Cu at (115.3, 134.6)
- added R7: 100, Footprints:R_LOAD, F.Cu at (187.4, 199.1)
- added R8: 100, Resistor_SMD:R_1206_3216Metric_Pad1.30x1.75mm_HandSolder, F.Cu at (167.9, 139.0)
- added S1: 1-1337445-0, Footprints:TE_1-1337445-0, F.Cu at (140.6, 98.2)
- added S2: NDI-04H-V, Footprints:NDI04HV, F.Cu at (146.2, 163.9)
- added SW1: SL19-121, Footprints:SL19121, F.Cu at (107.3, 100.9)
- added SW2: SL19-121, Footprints:SL19121, F.Cu at (162.5, 101.0)
- added SW3: SL19-121, Footprints:SL19121, F.Cu at (107.9, 159.0)
- added SW4: SL19-121, Footprints:SL19121, F.Cu at (162.8, 160.1)
- added TVS1: D_Zener, Footprints:SMFSeries_LTF, F.Cu at (115.0, 118.0)
- added TVS2: D_Zener, Footprints:SMFSeries_LTF, F.Cu at (167.9, 132.4)
- added TVS3: D_Zener, Footprints:SMFSeries_LTF, F.Cu at (115.3, 129.9)
- added TVS4: D_Zener, Footprints:SMFSeries_LTF, F.Cu at (167.7, 143.6)
Routing:
- net /V_IN+: track 0.00 -> 547.7 mm, vias 0 -> 1
- net V_G2: track 0.00 -> 112.0 mm, vias 0 -> 2
- net V_G1: track 0.00 -> 97.3 mm, vias 0 -> 3
- net V_G3: track 0.00 -> 96.6 mm, vias 0 -> 3
- net V_G4: track 0.00 -> 90.3 mm
- net /Drain_1: track 0.00 -> 60.8 mm, vias 0 -> 2
- net /Drain_4: track 0.00 -> 53.8 mm, vias 0 -> 2
- net /Drain_3: track 0.00 -> 51.0 mm
- net /Drain_2: track 0.00 -> 47.5 mm
- net /V_G: track 0.00 -> 25.2 mm
- net Net-(Q2-G): track 0.00 -> 16.6 mm
- net Net-(Q4-G): track 0.00 -> 16.5 mm
- net Net-(Q1-G): track 0.00 -> 14.8 mm
- net Net-(Q3-G): track 0.00 -> 14.3 mm
- net GND: vias 0 -> 12
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- added copper zone on B.Cu, net GND
- added copper zone on F.Cu, net GND
Other:
- board outline added: 150 x 150 mm
- board text added: "G1 G2 G3 G4"
- board text added: "LOAD_ON_1"
- board text added: "LOAD_ON_2"
- board text added: "LOAD_ON_3"
- board text added: "LOAD_ON_4"

Commit message: PCB final version
Parts:
- added REF**: Symbol_Radiation_Trefoil_15mm_Silkscreen, Radioactive_Symbol_KiCad9:Symbol_Radiation_Trefoil_15mm_Silkscreen, F.Cu at (141.1, 70.8)
- added REF**: ESD-Logo_6.6x6mm_SilkScreen, Symbol:ESD-Logo_6.6x6mm_SilkScreen, F.Cu at (187.8, 198.1)
