File: PCB design/GaN_Transistor_Test_Board.kicad_sch (KiCad schematic)
At the start: 17 parts, among them J1 Conn_01x01, J2 Conn_01x01, J3 Conn_01x01, J4 Conn_01x01, Q1 IGD70R500D2S

Commit message: PCB_rev1
Parts:
- removed J4: Conn_01x01, Footprints:CONN1_FCR7350R_CLF, symbol Connector_Generic:Conn_01x01
- removed TP1, TP2, TP3, TP4, TP5, TP6: TestPoint, symbol Connector:TestPoint
- added D2, D3, D4, G2, G3, G4: 1-1337445-0, Footprints:TE_1-1337445-0, symbol 1-1337445-0:1-1337445-0
- added H1, H2, H3, H4: MountingHole, MountingHole:MountingHole_4.3mm_M4, symbol Mechanical:MountingHole
- added Q2, Q3, Q4: IGD70R500D2S, Footprints:IFX-PG-TO252-3N-37-V1, symbol IGD70R500D2S:IGD70R500D2S
- added R3, R5, R7: 100, Footprints:R_LOAD, symbol Device:R
- added R4, R6, R8: 100, Resistor_SMD:R_1206_3216Metric_Pad1.30x1.75mm_HandSolder, symbol Device:R
- added S2: NDI-04H-V, Footprints:NDI04HV, symbol NDI-04H-V:NDI-04H-V
- added SW1, SW2, SW3, SW4: SL19-121, Footprints:SL19121, symbol 1-1337445-0:SL19-121
- added TVS2, TVS3, TVS4: D_Zener, Footprints:SMFSeries_LTF, symbol Device:D_Zener
- R1: value 680 -> 100; footprint (none) -> Footprints:R_LOAD
- R2: footprint Resistor_SMD:R_0805_2012Metric_Pad1.20x1.40mm_HandSolder -> Resistor_SMD:R_1206_3216Metric_Pad1.30x1.75mm_HandSolder
Connections:
- net GND: now also J2.1 (Pin_1), D2.SH3 (GND), D3.SH3 (GND), D4.SH3 (GND), G2.SH1 (GND), G3.SH1 (GND), G4.SH1 (GND), Q2.2 (S), Q3.2 (S), Q4.2 (S), TVS2.1 (K), TVS3.1 (K), TVS4.1 (K); no longer J3.1 (Pin_1)
- net Drain_1: now reaches Q1.3 (D), R1.2
- net Drain_1: now also SW1.3
- net V_G1: now reaches G1.1 (SIG), R2.2
- net V_G1: now also S2.8 (NO_1); no longer J2.1 (Pin_1)
- net V_IN+: now reaches D1.1 (SIG), J1.1 (Pin_1), R1.1
- net V_IN+: now also D2.1 (SIG), D3.1 (SIG), D4.1 (SIG), R3.1, R5.1, R7.1, SW1.2, SW2.2, SW3.2, SW4.2
- new net: Q2.1 (G), R4.1, TVS2.2 (A)
- new net: Q4.1 (G), R8.1, TVS4.2 (A)
- new net: Q3.1 (G), R6.1, TVS3.2 (A)
- new net Drain_2: Q2.3 (D), R3.2, SW2.3
- new net Drain_3: Q3.3 (D), R5.2, SW3.3
- new net Drain_4: Q4.3 (D), R7.2, SW4.3
- new net V_G: J3.1 (Pin_1), S2.1 (COM_1), S2.2 (COM_2), S2.3 (COM_3), S2.4 (COM_4)
- new net V_G2: G2.1 (SIG), R4.2, S2.7 (NO_2)
- new net V_G3: G3.1 (SIG), R6.2, S2.6 (NO_3)
- new net V_G4: G4.1 (SIG), R8.2, S2.5 (NO_4)
- no-connect marks 0 -> 4
Other:
- moved on the sheet: D1, G1, Q1, R1, R2, S1, TVS1
